File: hardware/calibrator.kicad_sch (KiCad schematic)
At the start: 17 parts, among them J1 BNC female, J2 JST 3-pin, SW1 ON-OFF-ON, SW2 push button, U1 ESP32-C3 SuperMini, U2 ADS1115 module, U3 SSD1306 OLED 128x64

Commit message: No VMID divider, crossed cable: the schematic and wiring diagram match the built unit
An ohmmeter check found nothing between A1 and 3.3 V or GND: the calibrator has no
VMID divider, and A1 floats until a pH board is connected. The divider added in
f99d40c is removed from the KiCad schematic, the wiring diagram and the READMEs.
Channel A is documented as valid only with a board connected, the divider as an
optional addition. The 50 MΩ series resistor is five 10 MΩ SMD in series.

The JST is numbered as built: 1 GND (through Rsh), 2 +5 V, 3 S. The pH board's P2 is
VCC, com, S, so the cable between them is crossed; the docs say to wire it by function.

Co-Authored-By: Claude Opus 5.5 <noreply@anthropic.com>
Parts:
- removed C1: 100n, symbol Device:C
- removed R6, R7: 10k, symbol Device:R
- R2: value 50M -> 50M (5x10M)
Connections:
- net +5V: now also J2.2 (Pin_2); no longer J2.1 (Pin_1)
- net BOARD_GND: now also J2.1 (Pin_1); no longer J2.2 (Pin_2)
Other:
- note added: "1. Power the ADS1115 and the OLED from 3.3 V, never from 5 V. 2. The simulator voltage E is measured BEFORE R2; the board input VIN is worked out from S. 3. Leakage: I = (VIN - E) / R2 after a two-point calibration with SW2 pressed. 4. The simulator floats and REF has no divider of its own: channel A is valid only with a pH board connected. 5. Optional, not fitted: 10k from 3.3 V and 10k to GND w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"
- note added: "J2 as built: 1 GND (through R5), 2 +5V, 3 S. P2 on the pH board is 1 VCC, 2 com, 3 S: the cable is crossed. Wire it by function and check it before power-up."
- note removed: "1. Power the ADS1115 and the OLED from 3.3 V, never from 5 V. 2. The simulator voltage E is measured BEFORE R2; the board input VIN is worked out from S. 3. Leakage: I = (VIN - E) / R2 after a two-point calibration with SW2 pressed. 4. The simulator floats: its reference REF is tied only to VMID (R6, R7) and to the BNC shield."
- note removed: "J2 to P2 of the pH board, straight cable: 1 +5V 2 GND (through R5) 3 S"
- note removed: "VMID = 1.65 V (R6, R7, C1) holds the floating simulator inside the ADS1115 input range."
