File: hardware/calibrator.kicad_sch (KiCad schematic)
At the start: 14 parts, among them J1 BNC female, J2 JST 3-pin, SW1 ON-OFF-ON, SW2 push button, U1 ESP32-C3 SuperMini, U2 ADS1115 module, U3 SSD1306 OLED 128x64

Commit message: Add USB supply measurement to schematic and documentation
Parts:
- added JP1: 5V / 3.3V, symbol Jumper:Jumper_3_Open
- added R6: 10K, symbol Device:R
- added R7: 15K, symbol Device:R
- added TP1: REF, symbol Connector:TestPoint
- added TP2: E, symbol Connector:TestPoint
- added TP3: VIN, symbol Connector:TestPoint
Connections:
- net +3V3: now also JP1.3 (B)
- net +5V: now also JP1.1 (A), R7.1; no longer J2.2 (Pin_2)
- net E: now also TP2.1
- net GND: now also R6.2
- net REF: now also TP1.1
- net VIN: now also TP3.1
- net at U1.4 (GPIO4): now also R6.1, R7.2
- new net BOARD_VCC: J2.2 (Pin_2), JP1.2 (C)
- no-connect marks 12 -> 11
Other:
- note added: "J2 as built: 1 GND (through R5), 2 supply (JP1: 5 V or 3.3 V), 3 S. P2 on the pH board is 1 VCC, 2 com, 3 S: the cable is crossed. Wire it by function and check it before power-up."
- note added: "Test pins: TP1 BNC shield (REF), TP2 BNC + before R2 (E), TP3 BNC + after R2 (VIN). TP3 is the high-impedance node: touch it only with an electrometer."
- note removed: "J2 as built: 1 GND (through R5), 2 +5V, 3 S. P2 on the pH board is 1 VCC, 2 com, 3 S: the cable is crossed. Wire it by function and check it before power-up."
